File: SiD-Touch/KiCad/ESP32-Touch_board/ESP32-Touch_board.kicad_pcb (KiCad board)
At the start: 2 copper layers, 43 x 43 mm, 47 parts, among them J1 Screw_Terminal_01x04, J2 TOUCH_PINS, J3 JUMPER 120R, J4 BUS_PINS, J5 PROG, Q1 BC817, Q2 BC817, U1 SN65HVD230, U2 XL1509-3.3, U3 ESP32-C3-MINI-1-N4

Commit message: touch02
Parts:
- added R16: 10k/R0603, Resistor_SMD:R_0603_1608Metric, F.Cu at (71.0, 112.0)
- added R17: 10k/R0603, Resistor_SMD:R_0603_1608Metric, F.Cu at (72.8, 112.0)
- moved J3 4.25 mm to (89.5, 125.6)
- moved R8 1.98 mm to (89.8, 122.8)
- moved R7 1.19 mm to (88.5, 112.4)
- moved D6 1.19 mm to (88.5, 116.9)
- moved D7 1.19 mm to (88.5, 114.7)
- moved R6 1.19 mm to (88.5, 119.2)
- moved R9 0.95 mm to (69.3, 112.0)
- moved G*** 0.85 mm to (59.5, 109.0)
- moved D8 0.83 mm to (67.6, 112.0)
- moved R15 0.36 mm to (74.5, 112.0)
- moved C1 0.33 mm to (76.2, 112.0)
- moved C2 0.27 mm to (77.9, 112.0)
- turned D5 to 0 degrees
Routing:
- net +3V3: track 0.00 -> 108.7 mm, vias 0 -> 7
- net TOUCH_1: track 0.00 -> 42.8 mm, vias 0 -> 1
- net TOUCH_2: track 0.00 -> 38.6 mm, vias 0 -> 1
- net RXDO: track 0.00 -> 35.7 mm, vias 0 -> 2
- net TOUCH_4: track 0.00 -> 28.4 mm, vias 0 -> 1
- net GPIO8: track 0.00 -> 28.1 mm, vias 0 -> 2
- net 1-WIRE: track 0.00 -> 26.5 mm, vias 0 -> 1
- net CAN_L: track 0.00 -> 26.1 mm, vias 0 -> 3
- net TXDO: track 0.00 -> 26.1 mm, vias 0 -> 2
- net SDA: track 0.00 -> 25.9 mm, vias 0 -> 1
- net TOUCH_3: track 0.00 -> 24.3 mm, vias 0 -> 1
- net CAN_H: track 0.00 -> 23.9 mm
- net TX_CAN: track 0.00 -> 23.8 mm, vias 0 -> 2
- net CHIP_PU: track 0.00 -> 22.9 mm, vias 0 -> 2
- net SCL: track 0.00 -> 22.7 mm, vias 0 -> 1
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- added copper zone on F.Cu, net +24V
- added copper zone on F.Cu, net +3V3
- added copper zone on B.Cu, net GND
- added copper zone on F.Cu, net GND
Other:
- board text added: "+24V"
- board text added: "CAN_H"
- board text added: "CAN_L"
