File: SiD-Touch/KiCad/ESP32-Touch_board/ESP32-Touch_board.kicad_sch (KiCad schematic)
At the start: 44 parts, among them J1 Screw_Terminal_01x04, J2 PROG, J3 JUMPER 120R, J4 TOUCH_PINS, J5 BUS_PINS, Q1 BC817, Q2 BC817, U1 ESP32-C3-MINI-1-N4, U2 XL1509-3.3, U3 SN65HVD230

Commit message: PCB cont
Parts:
- removed D2: SS34, Diode_SMD:D_SMA, symbol Device:D_Filled
- removed L2: ACT45B-510, symbol Device:L_Coupled
- added D4: 1N5819WS, Diode_SMD:D_SOD-323_HandSoldering, symbol Device:D_Schottky
- added L1: ACT45B-510, ACT45B:FIL_ACT45B-510-2P-TL003, symbol Device:L_Coupled_1423
- added R4, R5: 0k/R0603, Resistor_SMD:R_0603_1608Metric, symbol Device:R
- C1: renamed from C8; value 1uF/C0805 -> 10uF/C0805; footprint Capacitor_SMD:C_0805_2012Metric -> Capacitor_SMD:C_0603_1608Metric; JLCPCB C111768 -> C380314
- C10: renamed from C5; value 1uF/C0805 -> 10uF/C0805; footprint Capacitor_SMD:C_0805_2012Metric -> Capacitor_SMD:C_0603_1608Metric; JLCPCB C111768 -> C380314
- C8: renamed from C6; value 1uF/C0805 -> 10uF/C0805; footprint Capacitor_SMD:C_0805_2012Metric -> Capacitor_SMD:C_0603_1608Metric; JLCPCB C111768 -> C380314
- D1: footprint Diode_SMD:D_SMA -> Diode_SMD:D_SOD-323_HandSoldering
- J1: footprint (none) -> Connector_Phoenix_MC:PhoenixContact_MCV_1,5_4-G-3.81_1x04_P3.81mm_Vertical
- J2: renamed from J4; footprint (none) -> Connector_PinHeader_2.54mm:PinHeader_1x06_P2.54mm_Vertical
- J3: footprint (none) -> Jumper:SolderJumper-2_P1.3mm_Open_RoundedPad1.0x1.5mm
- J4: renamed from J5; footprint (none) -> Connector_PinHeader_2.54mm:PinHeader_1x06_P2.54mm_Vertical
- J5: renamed from J2; footprint (none) -> Connector_PinHeader_2.00mm:PinHeader_1x06_P2.00mm_Vertical
- L2: renamed from L1; value 47uH/2.5A -> 47uH/900mA; footprint Inductor_SMD:L_7.3x7.3_H4.5 -> Inductor_SMD:L_Sunlord_SWPA5040S; JLCPCB C436585 -> C142114
- U3: renamed from U1; footprint XCVR_ESP32-C3-MINI-1-N4 -> ESP32-C3-MINI-1-N4:XCVR_ESP32-C3-MINI-1-N4
- renumbered C7 to C2, C1 to C3, C2 to C4, C9 to C5, C10 to C6, C3 to C7, C4 to C9, D5 to D2, D6 to D3, D4 to D5, D7 to D6, D8 to D7, D3 to D8, R8 to R1, R1 to R10, R6 to R11, R7 to R12, R4 to R13, R5 to R14, R3 to R15, R12 to R2, R13 to R3, R10 to R6, R11 to R7, R9 to R8, R2 to R9, U3 to U1
Connections:
- net CAN_H: now also L1.4, R4.1
- net CAN_L: now also L1.3, R5.2
- net GND: now also D4.2 (A)
- net at U1.6 (CANL): now also L1.2, R5.1
- net at U1.7 (CANH): now also L1.1, R4.2
- net at L2.1, U2.2 (OUT): now also D4.1 (K)

Commit message: touch02
Parts:
- added R16, R17: 10k/R0603, Resistor_SMD:R_0603_1608Metric, symbol Device:R
Connections:
- net +3V3: now also R16.2, R17.2
- net SCL: now also R16.1
- net SDA: now also R17.1
Changed lines of the file:
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@@
+    (stroke (width 0) (type default))
+  )
+  (wire (pts (xy 151.13 165.1) (xy 151.13 168.275))
     (stroke (width 0) (type default))
   )
@@
     (stroke (width 0) (type default))
   )
+  (wire (pts (xy 160.655 179.705) (xy 160.655 175.895))
+    (stroke (width 0) (type default))
+  )
   (wire (pts (xy 114.935 177.165) (xy 120.015 177.165))
     (stroke (width 0) (type default))
@@
     (stroke (width 0) (type default))
   )
+  (wire (pts (xy 151.13 179.705) (xy 151.13 175.895))
+    (stroke (width 0) (type default))
+  )
   (wire (pts (xy 255.27 48.895) (xy 255.27 50.8))
     (stroke (width 0) (type default))
@@
   )
   (wire (pts (xy 147.32 71.755) (xy 147.32 74.93))
+    (stroke (width 0) (type default))
+  )
+  (wire (pts (xy 160.655 165.1) (xy 160.655 168.275))
     (stroke (width 0) (type default))
   )
@@
     )
   )
+  (global_label "SDA" (shape input) (at 160.655 179.705 270) (fields_autoplaced)
+    (effects (font (size 1.27 1.27)) (justify right))
+    (property "Intersheetrefs" "${INTERSHEET_REFS}" (at 160.655 186.1789 90)
+      (effects (font (size 1.27 1.27)) (justify right) hide)
+    )
+  )
   (global_label "SDA" (shape input) (at 197.485 69.85 180) (fields_autoplaced)
     (effects (font (size 1.27 1.27)) (justify right))
@@
     (property "Intersheetrefs" "${INTERSHEET_REFS}" (at 251.1606 72.39 0)
       (effects (font (size 1.27 1.27)) (justify left) hide)
+    )
+  )
+  (global_label "SCL" (shape input) (at 151.13 179.705 270) (fields_autoplaced)
+    (effects (font (size 1.27 1.27)) (justify right))
+    (property "Intersheetrefs" "${INTERSHEET_REFS}" (at 151.13 186.1184 90)
+      (effects (font (size 1.27 1.27)) (justify right) hide)
     )
   )
@@
         (path "/e63e39d7-6ac0-4ffd-8aa3-1841a4541b55"
           (reference "R5") (unit 1)
+        )
+      )
+    )
+  )
+  (symbol (lib_id "power:+3.3V") (at 151.13 165.1 0) (unit 1)
+    (in_bom yes) (on_board yes) (dnp no)
+    (property "Reference" "#PWR033" (at 151.13 168.91 0)
+      (effects (font (size 1.27 1.27)) hide)
+    )
+    (property "Value" "+3.3V" (at 151.511 160.7058 0)
+      (effects (font (size 1.27 1.27)))
+    )
+    (property "Footprint" "" (at 151.13 165.1 0)
+      (effects (font (size 1.27 1.27)) hide)
+    )
+    (property "Datasheet" "" (at 151.13 165.1 0)
+      (effects (font (size 1.27 1.27)) hide)
+    )
+    (pin "1")
+    (instances
+      (project "ESP32-Touch_board"
+        (path "/d70a78be-4422-4416-98f1-757de7245ee7"
+          (reference "#PWR033") (unit 1)
+        )
+      )
+      (project "boneIO - input WT32"
+        (path "/e63e39d7-6ac0-4ffd-8aa3-1841a4541b55"
+          (reference "#PWR0234") (unit 1)
         )
       )
@@
     )
   )
+  (symbol (lib_id "Device:R") (at 160.655 172.085 180) (unit 1)
+    (in_bom yes) (on_board yes) (dnp no)
+    (property "Reference" "R17" (at 163.195 170.815 90)
+      (effects (font (size 1 1)) (justify left))
+    )
+    (property "Value" "10k/R0603" (at 165.1 167.64 90)
+      (effects (font (size 1 1)) (justify left))
+    )
+    (property "Footprint" "Resistor_SMD:R_0603_1608Metric" (at 162.433 172.085 90)
+      (effects (font (size 1.27 1.27)) hide)
+    )
+    (property "Datasheet" "~" (at 160.655 172.085 0)
+      (effects (font (size 1.27 1.27)) hide)
+    )
+    (property "JLCPCB" "C25804" (at 167.005 171.45 90)
+      (effects (font (size 1 1)))
+    )
+    (pin "1")
+    (pin "2")
+    (instances
+      (project "ESP32-Touch_board"
+        (path "/d70a78be-4422-4416-98f1-757de7245ee7"
+          (reference "R17") (unit 1)
+        )
+      )
+      (project "SIGMA Switch v0.2"
+        (path "/e63e39d7-6ac0-4ffd-8aa3-1841a4541b55"
+          (reference "R9") (unit 1)
+        )
+      )
+    )
+  )
   (symbol (lib_id "Device:Fuse") (at 52.07 57.15 270) (unit 1)
     (in_bom yes) (on_board yes) (dnp no)
@@
     )
   )
+  (symbol (lib_id "Device:R") (at 151.13 172.085 180) (unit 1)
+    (in_bom yes) (on_board yes) (dnp no)
+    (property "Reference" "R16" (at 153.67 170.815 90)
+      (effects (font (size 1 1)) (justify left))
+    )
+    (property "Value" "10k/R0603" (at 155.575 167.64 90)
+      (effects (font (size 1 1)) (justify left))
+    )
+    (property "Footprint" "Resistor_SMD:R_0603_1608Metric" (at 152.908 172.085 90)
+      (effects (font (size 1.27 1.27)) hide)
+    )
+    (property "Datasheet" "~" (at 151.13 172.085 0)
+      (effects (font (size 1.27 1.27)) hide)
+    )
+    (property "JLCPCB" "C25804" (at 157.48 171.45 90)
+      (effects (font (size 1 1)))
+    )
+    (pin "1")
+    (pin "2")
+    (instances
+      (project "ESP32-Touch_board"
+        (path "/d70a78be-4422-4416-98f1-757de7245ee7"
+          (reference "R16") (unit 1)
+        )
+      )
+      (project "SIGMA Switch v0.2"
+        (path "/e63e39d7-6ac0-4ffd-8aa3-1841a4541b55"
+          (reference "R9") (unit 1)
+        )
+      )
+    )
+  )
   (symbol (lib_id "Device:C_Polarized") (at 73.66 66.04 0) (unit 1)
     (in_bom yes) (on_board yes) (dnp no)
@@
         )
       )
+    )
+  )
+  (symbol (lib_id "power:+3.3V") (at 160.655 165.1 0) (unit 1)
+    (in_bom yes) (on_board yes) (dnp no)
+    (property "Reference" "#PWR034" (at 160.655 168.91 0)
+      (effects (font (size 1.27 1.27)) hide)
+    )
+    (property "Value" "+3.3V" (at 161.036 160.7058 0)
+      (effects (font (size 1.27 1.27)))
+    )
+    (property "Footprint" "" (at 160.655 165.1 0)
+      (effects (font (size 1.27 1.27)) hide)
+    )
+    (property "Datasheet" "" (at 160.655 165.1 0)
+      (effects (font (size 1.27 1.27)) hide)
+    )
+    (pin "1")
+    (instances
+      (project "ESP32-Touch_board"
+        (path "/d70a78be-4422-4416-98f1-757de7245ee7"
+          (reference "#PWR034") (unit 1)
+        )
+      )
+      (project "boneIO - input WT32"
+        (path "/e63e39d7-6ac0-4ffd-8aa3-1841a4541b55"
+          (reference "#PWR0234") (unit 1)
+        )
+      )
